Commit message: add hexapod.urdf file

File: urdf/hexapod.urdf (robot description, URDF)
Before this commit: robot hexapod, 7 links, 6 joints
Links:
- added link leg1_pitch_1, mass 0.7; collision cylinder length=0.14 radius=0.025; visual cylinder length=0.14 radius=0.025
- added link leg1_pitch_2, mass 0.8; collision cylinder length=0.16 radius=0.025; visual cylinder length=0.16 radius=0.025
- added link leg1_pitch_3, mass 0.7; collision cylinder length=0.14 radius=0.025; visual cylinder length=0.14 radius=0.025
- added link leg1_stick, mass 0.2; collision cylinder length=0.01 radius=0.065; visual cylinder length=0.01 radius=0.065
- added link leg2_pitch_1, mass 0.7; collision cylinder length=0.14 radius=0.025; visual cylinder length=0.14 radius=0.025
- added link leg2_pitch_2, mass 0.8; collision cylinder length=0.16 radius=0.025; visual cylinder length=0.16 radius=0.025
- added link leg2_pitch_3, mass 0.7; collision cylinder length=0.14 radius=0.025; visual cylinder length=0.14 radius=0.025
- added link leg2_stick, mass 0.2; collision cylinder length=0.01 radius=0.065; visual cylinder length=0.01 radius=0.065
- added link leg3_pitch_1, mass 0.7; collision cylinder length=0.14 radius=0.025; visual cylinder length=0.14 radius=0.025
- added link leg3_pitch_2, mass 0.8; collision cylinder length=0.16 radius=0.025; visual cylinder length=0.16 radius=0.025
- added link leg3_pitch_3, mass 0.7; collision cylinder length=0.14 radius=0.025; visual cylinder length=0.14 radius=0.025
- added link leg3_stick, mass 0.2; collision cylinder length=0.01 radius=0.065; visual cylinder length=0.01 radius=0.065
- added link leg4_pitch_1, mass 0.7; collision cylinder length=0.14 radius=0.025; visual cylinder length=0.14 radius=0.025
- added link leg4_pitch_2, mass 0.8; collision cylinder length=0.16 radius=0.025; visual cylinder length=0.16 radius=0.025
- added link leg4_pitch_3, mass 0.7; collision cylinder length=0.14 radius=0.025; visual cylinder length=0.14 radius=0.025
- added link leg4_stick, mass 0.2; collision cylinder length=0.01 radius=0.065; visual cylinder length=0.01 radius=0.065
- added link leg5_pitch_1, mass 0.7; collision cylinder length=0.14 radius=0.025; visual cylinder length=0.14 radius=0.025
- added link leg5_pitch_2, mass 0.8; collision cylinder length=0.16 radius=0.025; visual cylinder length=0.16 radius=0.025
- added link leg5_pitch_3, mass 0.7; collision cylinder length=0.14 radius=0.025; visual cylinder length=0.14 radius=0.025
- added link leg5_stick, mass 0.2; collision cylinder length=0.01 radius=0.065; visual cylinder length=0.01 radius=0.065
- added link leg6_pitch_1, mass 0.7; collision cylinder length=0.14 radius=0.025; visual cylinder length=0.14 radius=0.025
- added link leg6_pitch_2, mass 0.8; collision cylinder length=0.16 radius=0.025; visual cylinder length=0.16 radius=0.025
- added link leg6_pitch_3, mass 0.7; collision cylinder length=0.14 radius=0.025; visual cylinder length=0.14 radius=0.025
- added link leg6_stick, mass 0.2; collision cylinder length=0.01 radius=0.065; visual cylinder length=0.01 radius=0.065
- link base: mass 1 -> 2
- link leg1_roll: mass 1 -> 0.45; geometry collision cylinder length=0.09 radius=0.025; visual cylinder length=0.09 radius=0.025
- link leg2_roll: mass 1 -> 0.45; geometry collision cylinder length=0.09 radius=0.025; visual cylinder length=0.09 radius=0.025
- link leg3_roll: mass 1 -> 0.45; geometry collision cylinder length=0.09 radius=0.025; visual cylinder length=0.09 radius=0.025
- link leg4_roll: mass 1 -> 0.45; geometry collision cylinder length=0.09 radius=0.025; visual cylinder length=0.09 radius=0.025
- link leg5_roll: mass 1 -> 0.45; geometry collision cylinder length=0.09 radius=0.025; visual cylinder length=0.09 radius=0.025
- link leg6_roll: mass 1 -> 0.45; geometry collision cylinder length=0.09 radius=0.025; visual cylinder length=0.09 radius=0.025
Joints:
- added joint leg1_joint_pitch_1: type revolute, parent leg1_roll, child leg1_pitch_1, origin xyz=0.09 0 0 rpy=1.570796 0 0, axis 0 0 1, limit lower=-4.71238898 upper=1.570796 effort=300 velocity=1
- added joint leg1_joint_pitch_2: type revolute, parent leg1_pitch_1, child leg1_pitch_2, origin xyz=0.14 0 0 rpy=0 0 -1.570796, axis 0 0 1, limit lower=-4.71238898 upper=3.141592653 effort=300 velocity=1
- added joint leg1_joint_pitch_3: type revolute, parent leg1_pitch_2, child leg1_pitch_3, origin xyz=0.16 0 0 rpy=0 0 0, axis 0 0 1, limit lower=-4.71238898 upper=1.57075 effort=300 velocity=1
- added joint leg1_joint_stick: type revolute, parent leg1_pitch_3, child leg1_stick, origin xyz=0.14 0 0 rpy=0 0 0, axis 1 1 1, limit lower=-1.57075 upper=1.57075 effort=300 velocity=1
- added joint leg2_joint_pitch_1: type revolute, parent leg2_roll, child leg2_pitch_1, origin xyz=0.09 0 0 rpy=1.570796 0 0, axis 0 0 1, limit lower=-4.71238898 upper=1.570796 effort=300 velocity=1
- added joint leg2_joint_pitch_2: type revolute, parent leg2_pitch_1, child leg2_pitch_2, origin xyz=0.14 0 0 rpy=0 0 -1.570796, axis 0 0 1, limit lower=-4.71238898 upper=3.141592653 effort=300 velocity=1
- added joint leg2_joint_pitch_3: type revolute, parent leg2_pitch_2, child leg2_pitch_3, origin xyz=0.16 0 0 rpy=0 0 0, axis 0 0 1, limit lower=-4.71238898 upper=1.57075 effort=300 velocity=1
- added joint leg2_joint_stick: type revolute, parent leg2_pitch_3, child leg2_stick, origin xyz=0.14 0 0 rpy=0 0 0, axis 1 1 1, limit lower=-1.57075 upper=1.57075 effort=300 velocity=1
- added joint leg3_joint_pitch_1: type revolute, parent leg3_roll, child leg3_pitch_1, origin xyz=0.09 0 0 rpy=1.570796 0 0, axis 0 0 1, limit lower=-4.71238898 upper=1.570796 effort=300 velocity=1
- added joint leg3_joint_pitch_2: type revolute, parent leg3_pitch_1, child leg3_pitch_2, origin xyz=0.14 0 0 rpy=0 0 -1.570796, axis 0 0 1, limit lower=-4.71238898 upper=3.141592653 effort=300 velocity=1
- added joint leg3_joint_pitch_3: type revolute, parent leg3_pitch_2, child leg3_pitch_3, origin xyz=0.16 0 0 rpy=0 0 0, axis 0 0 1, limit lower=-4.71238898 upper=1.57075 effort=300 velocity=1
- added joint leg3_joint_stick: type revolute, parent leg3_pitch_3, child leg3_stick, origin xyz=0.14 0 0 rpy=0 0 0, axis 1 1 1, limit lower=-1.57075 upper=1.57075 effort=300 velocity=1
- added joint leg4_joint_pitch_1: type revolute, parent leg4_roll, child leg4_pitch_1, origin xyz=0.09 0 0 rpy=1.570796 0 0, axis 0 0 1, limit lower=-4.71238898 upper=1.570796 effort=300 velocity=1
- added joint leg4_joint_pitch_2: type revolute, parent leg4_pitch_1, child leg4_pitch_2, origin xyz=0.14 0 0 rpy=0 0 -1.570796, axis 0 0 1, limit lower=-4.71238898 upper=3.141592653 effort=300 velocity=1
- added joint leg4_joint_pitch_3: type revolute, parent leg4_pitch_2, child leg4_pitch_3, origin xyz=0.16 0 0 rpy=0 0 0, axis 0 0 1, limit lower=-4.71238898 upper=1.57075 effort=300 velocity=1
- added joint leg4_joint_stick: type revolute, parent leg4_pitch_3, child leg4_stick, origin xyz=0.14 0 0 rpy=0 0 0, axis 1 1 1, limit lower=-1.57075 upper=1.57075 effort=300 velocity=1
- added joint leg5_joint_pitch_1: type revolute, parent leg5_roll, child leg5_pitch_1, origin xyz=0.09 0 0 rpy=1.570796 0 0, axis 0 0 1, limit lower=-4.71238898 upper=1.570796 effort=300 velocity=1
- added joint leg5_joint_pitch_2: type revolute, parent leg5_pitch_1, child leg5_pitch_2, origin xyz=0.14 0 0 rpy=0 0 -1.570796, axis 0 0 1, limit lower=-4.71238898 upper=3.141592653 effort=300 velocity=1
- added joint leg5_joint_pitch_3: type revolute, parent leg5_pitch_2, child leg5_pitch_3, origin xyz=0.16 0 0 rpy=0 0 0, axis 0 0 1, limit lower=-4.71238898 upper=1.57075 effort=300 velocity=1
- added joint leg5_joint_stick: type revolute, parent leg5_pitch_3, child leg5_stick, origin xyz=0.14 0 0 rpy=0 0 0, axis 1 1 1, limit lower=-1.57075 upper=1.57075 effort=300 velocity=1
- added joint leg6_joint_pitch_1: type revolute, parent leg6_roll, child leg6_pitch_1, origin xyz=0.09 0 0 rpy=1.570796 0 0, axis 0 0 1, limit lower=-4.71238898 upper=1.570796 effort=300 velocity=1
- added joint leg6_joint_pitch_2: type revolute, parent leg6_pitch_1, child leg6_pitch_2, origin xyz=0.14 0 0 rpy=0 0 -1.570796, axis 0 0 1, limit lower=-4.71238898 upper=3.141592653 effort=300 velocity=1
- added joint leg6_joint_pitch_3: type revolute, parent leg6_pitch_2, child leg6_pitch_3, origin xyz=0.16 0 0 rpy=0 0 0, axis 0 0 1, limit lower=-4.71238898 upper=1.57075 effort=300 velocity=1
- added joint leg6_joint_stick: type revolute, parent leg6_pitch_3, child leg6_stick, origin xyz=0.14 0 0 rpy=0 0 0, axis 1 1 1, limit lower=-1.57075 upper=1.57075 effort=300 velocity=1

Commit message: add env file

File: urdf/hexapod.urdf (robot description, URDF)
Before this commit: robot hexapod, 31 links, 30 joints
Joints:
- joint leg1_joint_roll: limit (none) -> lower=-1.570796 upper=1.570796 effort=300 velocity=1
- joint leg2_joint_roll: limit (none) -> lower=-1.570796 upper=1.570796 effort=300 velocity=1
- joint leg3_joint_roll: limit (none) -> lower=-1.570796 upper=1.570796 effort=300 velocity=1
- joint leg4_joint_roll: limit (none) -> lower=-1.570796 upper=1.570796 effort=300 velocity=1
- joint leg5_joint_roll: limit (none) -> lower=-1.570796 upper=1.570796 effort=300 velocity=1
- joint leg6_joint_roll: limit (none) -> lower=-1.570796 upper=1.570796 effort=300 velocity=1

Commit message: 5.11

File: urdf/hexapod.urdf (robot description, URDF)
Before this commit: robot hexapod, 31 links, 30 joints
Joints:
- joint leg1_joint_pitch_1: limit lower=-4.71238898 upper=1.570796 effort=300 velocity=1 -> lower=-1.570796 upper=1.570796 effort=300 velocity=1; origin xyz=0.09 0 0 rpy=1.570796 0 0 -> xyz=0.09 0 0 rpy=1.5708 0 0
- joint leg1_joint_pitch_2: limit lower=-4.71238898 upper=3.141592653 effort=300 velocity=1 -> lower=-0.7854 upper=1.570796 effort=300 velocity=1; origin xyz=0.14 0 0 rpy=0 0 -1.570796 -> xyz=0.14 0 0 rpy=0 0 -1.5708
- joint leg1_joint_pitch_3: limit lower=-4.71238898 upper=1.57075 effort=300 velocity=1 -> lower=-1.570796 upper=1.570796 effort=300 velocity=1
- joint leg1_joint_roll: limit lower=-1.570796 upper=1.570796 effort=300 velocity=1 -> lower=-0.7854 upper=1.3090 effort=300 velocity=1
- joint leg1_joint_stick: limit lower=-1.57075 upper=1.57075 effort=300 velocity=1 -> lower=-0.08727 upper=0.08727 effort=300 velocity=1
- joint leg2_joint_pitch_1: limit lower=-4.71238898 upper=1.570796 effort=300 velocity=1 -> lower=-1.570796 upper=1.570796 effort=300 velocity=1; origin xyz=0.09 0 0 rpy=1.570796 0 0 -> xyz=0.09 0 0 rpy=1.5708 0 0
- joint leg2_joint_pitch_2: limit lower=-4.71238898 upper=3.141592653 effort=300 velocity=1 -> lower=-0.7854 upper=1.570796 effort=300 velocity=1; origin xyz=0.14 0 0 rpy=0 0 -1.570796 -> xyz=0.14 0 0 rpy=0 0 -1.5708
- joint leg2_joint_pitch_3: limit lower=-4.71238898 upper=1.57075 effort=300 velocity=1 -> lower=-1.570796 upper=1.570796 effort=300 velocity=1
- joint leg2_joint_roll: limit lower=-1.570796 upper=1.570796 effort=300 velocity=1 -> lower=-0.7854 upper=1.3090 effort=300 velocity=1; origin xyz=0 0.18 0 rpy=0 0 1.57 -> xyz=0 0.18 0 rpy=0 0 1.5708
- joint leg2_joint_stick: limit lower=-1.57075 upper=1.57075 effort=300 velocity=1 -> lower=-0.08727 upper=0.08727 effort=300 velocity=1
- joint leg3_joint_pitch_1: limit lower=-4.71238898 upper=1.570796 effort=300 velocity=1 -> lower=-1.570796 upper=1.570796 effort=300 velocity=1; origin xyz=0.09 0 0 rpy=1.570796 0 0 -> xyz=0.09 0 0 rpy=1.5708 0 0
- joint leg3_joint_pitch_2: limit lower=-4.71238898 upper=3.141592653 effort=300 velocity=1 -> lower=-0.7854 upper=1.570796 effort=300 velocity=1; origin xyz=0.14 0 0 rpy=0 0 -1.570796 -> xyz=0.14 0 0 rpy=0 0 -1.5708
- joint leg3_joint_pitch_3: limit lower=-4.71238898 upper=1.57075 effort=300 velocity=1 -> lower=-1.570796 upper=1.570796 effort=300 velocity=1
- joint leg3_joint_roll: limit lower=-1.570796 upper=1.570796 effort=300 velocity=1 -> lower=-0.7854 upper=1.3090 effort=300 velocity=1
- joint leg3_joint_stick: limit lower=-1.57075 upper=1.57075 effort=300 velocity=1 -> lower=-0.08727 upper=0.08727 effort=300 velocity=1
- joint leg4_joint_pitch_1: limit lower=-4.71238898 upper=1.570796 effort=300 velocity=1 -> lower=-1.570796 upper=1.570796 effort=300 velocity=1; origin xyz=0.09 0 0 rpy=1.570796 0 0 -> xyz=0.09 0 0 rpy=1.5708 0 0
- joint leg4_joint_pitch_2: limit lower=-4.71238898 upper=3.141592653 effort=300 velocity=1 -> lower=-0.7854 upper=1.570796 effort=300 velocity=1; origin xyz=0.14 0 0 rpy=0 0 -1.570796 -> xyz=0.14 0 0 rpy=0 0 -1.5708
- joint leg4_joint_pitch_3: limit lower=-4.71238898 upper=1.57075 effort=300 velocity=1 -> lower=-1.570796 upper=1.570796 effort=300 velocity=1
- joint leg4_joint_roll: limit lower=-1.570796 upper=1.570796 effort=300 velocity=1 -> lower=-0.7854 upper=1.3090 effort=300 velocity=1
- joint leg4_joint_stick: limit lower=-1.57075 upper=1.57075 effort=300 velocity=1 -> lower=-0.08727 upper=0.08727 effort=300 velocity=1
- joint leg5_joint_pitch_1: limit lower=-4.71238898 upper=1.570796 effort=300 velocity=1 -> lower=-1.570796 upper=1.570796 effort=300 velocity=1; origin xyz=0.09 0 0 rpy=1.570796 0 0 -> xyz=0.09 0 0 rpy=1.5708 0 0
- joint leg5_joint_pitch_2: limit lower=-4.71238898 upper=3.141592653 effort=300 velocity=1 -> lower=-0.7854 upper=1.570796 effort=300 velocity=1; origin xyz=0.14 0 0 rpy=0 0 -1.570796 -> xyz=0.14 0 0 rpy=0 0 -1.5708
- joint leg5_joint_pitch_3: limit lower=-4.71238898 upper=1.57075 effort=300 velocity=1 -> lower=-1.570796 upper=1.570796 effort=300 velocity=1
- joint leg5_joint_roll: limit lower=-1.570796 upper=1.570796 effort=300 velocity=1 -> lower=-0.7854 upper=1.3090 effort=300 velocity=1; origin xyz=0 -0.18 0 rpy=0 0 -1.57 -> xyz=0 -0.18 0 rpy=0 0 -1.5708
- joint leg5_joint_stick: limit lower=-1.57075 upper=1.57075 effort=300 velocity=1 -> lower=-0.08727 upper=0.08727 effort=300 velocity=1
- joint leg6_joint_pitch_1: limit lower=-4.71238898 upper=1.570796 effort=300 velocity=1 -> lower=-1.570796 upper=1.570796 effort=300 velocity=1; origin xyz=0.09 0 0 rpy=1.570796 0 0 -> xyz=0.09 0 0 rpy=1.5708 0 0
- joint leg6_joint_pitch_2: limit lower=-4.71238898 upper=3.141592653 effort=300 velocity=1 -> lower=-0.7854 upper=1.570796 effort=300 velocity=1; origin xyz=0.14 0 0 rpy=0 0 -1.570796 -> xyz=0.14 0 0 rpy=0 0 -1.5708
- joint leg6_joint_pitch_3: limit lower=-4.71238898 upper=1.57075 effort=300 velocity=1 -> lower=-1.570796 upper=1.570796 effort=300 velocity=1
- joint leg6_joint_roll: limit lower=-1.570796 upper=1.570796 effort=300 velocity=1 -> lower=-0.7854 upper=1.3090 effort=300 velocity=1
- joint leg6_joint_stick: limit lower=-1.57075 upper=1.57075 effort=300 velocity=1 -> lower=-0.08727 upper=0.08727 effort=300 velocity=1
