Commit message: 5.18

File: urdf/new_hexapod.urdf (robot description, URDF)
Before this commit: robot hexapod, 31 links, 30 joints
Links:
- link base: mass 1.8 -> 6.107
- link leg1_pitch_1: mass 0.7 -> 0.275
- link leg1_pitch_2: mass 0.8 -> 0.314
- link leg1_pitch_3: mass 0.7 -> 0.275
- link leg1_roll: mass 0.45 -> 0.177
- link leg1_stick: mass 0.2 -> 0.133; geometry collision cylinder length=0.01 radius=0.065; visual cylinder length=0.01 radius=0.065
- link leg2_pitch_1: mass 0.7 -> 0.275
- link leg2_pitch_2: mass 0.8 -> 0.314
- link leg2_pitch_3: mass 0.7 -> 0.275
- link leg2_roll: mass 0.45 -> 0.177
- link leg2_stick: mass 0.2 -> 0.133; geometry collision cylinder length=0.01 radius=0.065; visual cylinder length=0.01 radius=0.065
- link leg3_pitch_1: mass 0.7 -> 0.275
- link leg3_pitch_2: mass 0.8 -> 0.314
- link leg3_pitch_3: mass 0.7 -> 0.275
- link leg3_roll: mass 0.45 -> 0.177
- link leg3_stick: mass 0.2 -> 0.133; geometry collision cylinder length=0.01 radius=0.065; visual cylinder length=0.01 radius=0.065
- link leg4_pitch_1: mass 0.7 -> 0.275
- link leg4_pitch_2: mass 0.8 -> 0.314
- link leg4_pitch_3: mass 0.7 -> 0.275
- link leg4_roll: mass 0.45 -> 0.177
- link leg4_stick: mass 0.2 -> 0.133; geometry collision cylinder length=0.01 radius=0.065; visual cylinder length=0.01 radius=0.065
- link leg5_pitch_1: mass 0.7 -> 0.275
- link leg5_pitch_2: mass 0.8 -> 0.314
- link leg5_pitch_3: mass 0.7 -> 0.275
- link leg5_roll: mass 0.45 -> 0.177
- link leg5_stick: mass 0.2 -> 0.133; geometry collision cylinder length=0.01 radius=0.065; visual cylinder length=0.01 radius=0.065
- link leg6_pitch_1: mass 0.7 -> 0.275
- link leg6_pitch_2: mass 0.8 -> 0.314
- link leg6_pitch_3: mass 0.7 -> 0.275
- link leg6_roll: mass 0.45 -> 0.177
- link leg6_stick: mass 0.2 -> 0.133; geometry collision cylinder length=0.01 radius=0.065; visual cylinder length=0.01 radius=0.065
Joints:
- joint leg1_joint_pitch_1: limit lower=-1.570796 upper=1.570796 effort=300 velocity=1 -> lower=-1.570796 upper=1.570796 effort=300 velocity=3
- joint leg1_joint_pitch_2: limit lower=-0.7854 upper=1.570796 effort=300 velocity=1 -> lower=-0.7854 upper=1.570796 effort=300 velocity=3
- joint leg1_joint_pitch_3: limit lower=-1.570796 upper=1.570796 effort=300 velocity=1 -> lower=-1.570796 upper=1.570796 effort=300 velocity=3
- joint leg1_joint_roll: limit lower=-0.7854 upper=1.3090 effort=300 velocity=1 -> lower=-0.7854 upper=1.3090 effort=300 velocity=3
- joint leg1_joint_stick: axis 0 0 1 -> 1 1 1; type fixed -> revolute
- joint leg2_joint_pitch_1: limit lower=-1.570796 upper=1.570796 effort=300 velocity=1 -> lower=-1.570796 upper=1.570796 effort=300 velocity=3
- joint leg2_joint_pitch_2: limit lower=-0.7854 upper=1.570796 effort=300 velocity=1 -> lower=-0.7854 upper=1.570796 effort=300 velocity=3
- joint leg2_joint_pitch_3: limit lower=-1.570796 upper=1.570796 effort=300 velocity=1 -> lower=-1.570796 upper=1.570796 effort=300 velocity=3
- joint leg2_joint_roll: limit lower=-0.7854 upper=1.3090 effort=300 velocity=1 -> lower=-0.7854 upper=1.3090 effort=300 velocity=3
- joint leg2_joint_stick: axis 0 0 1 -> 1 1 1; limit lower=-0.01 upper=0.01 effort=300 velocity=1 -> lower=-0.08 upper=0.08 effort=300 velocity=1
- joint leg3_joint_pitch_1: limit lower=-1.570796 upper=1.570796 effort=300 velocity=1 -> lower=-1.570796 upper=1.570796 effort=300 velocity=3
- joint leg3_joint_pitch_2: limit lower=-0.7854 upper=1.570796 effort=300 velocity=1 -> lower=-0.7854 upper=1.570796 effort=300 velocity=3
- joint leg3_joint_pitch_3: limit lower=-1.570796 upper=1.570796 effort=300 velocity=1 -> lower=-1.570796 upper=1.570796 effort=300 velocity=3
- joint leg3_joint_roll: limit lower=-0.7854 upper=1.3090 effort=300 velocity=1 -> lower=-0.7854 upper=1.3090 effort=300 velocity=3
- joint leg3_joint_stick: axis 0 0 1 -> 1 1 1; limit lower=-0.01 upper=0.01 effort=300 velocity=1 -> lower=-0.08 upper=0.08 effort=300 velocity=1
- joint leg4_joint_pitch_1: limit lower=-1.570796 upper=1.570796 effort=300 velocity=1 -> lower=-1.570796 upper=1.570796 effort=300 velocity=3
- joint leg4_joint_pitch_2: limit lower=-0.7854 upper=1.570796 effort=300 velocity=1 -> lower=-0.7854 upper=1.570796 effort=300 velocity=3
- joint leg4_joint_pitch_3: limit lower=-1.570796 upper=1.570796 effort=300 velocity=1 -> lower=-1.570796 upper=1.570796 effort=300 velocity=3
- joint leg4_joint_roll: limit lower=-0.7854 upper=1.3090 effort=300 velocity=1 -> lower=-0.7854 upper=1.3090 effort=300 velocity=3
- joint leg4_joint_stick: axis 0 0 1 -> 1 1 1; limit lower=-0.01 upper=0.01 effort=300 velocity=1 -> lower=-0.08 upper=0.08 effort=300 velocity=1
- joint leg5_joint_pitch_1: limit lower=-1.570796 upper=1.570796 effort=300 velocity=1 -> lower=-1.570796 upper=1.570796 effort=300 velocity=3
- joint leg5_joint_pitch_2: limit lower=-0.7854 upper=1.570796 effort=300 velocity=1 -> lower=-0.7854 upper=1.570796 effort=300 velocity=3
- joint leg5_joint_pitch_3: limit lower=-1.570796 upper=1.570796 effort=300 velocity=1 -> lower=-1.570796 upper=1.570796 effort=300 velocity=3
- joint leg5_joint_roll: limit lower=-0.7854 upper=1.3090 effort=300 velocity=1 -> lower=-0.7854 upper=1.3090 effort=300 velocity=3
- joint leg5_joint_stick: axis 0 0 1 -> 1 1 1; limit lower=-0.01 upper=0.01 effort=300 velocity=1 -> lower=-0.08727 upper=0.08727 effort=300 velocity=1
- joint leg6_joint_pitch_1: limit lower=-1.570796 upper=1.570796 effort=300 velocity=1 -> lower=-1.570796 upper=1.570796 effort=300 velocity=3
- joint leg6_joint_pitch_2: limit lower=-0.7854 upper=1.570796 effort=300 velocity=1 -> lower=-0.7854 upper=1.570796 effort=300 velocity=3
- joint leg6_joint_pitch_3: limit lower=-1.570796 upper=1.570796 effort=300 velocity=1 -> lower=-1.570796 upper=1.570796 effort=300 velocity=3
- joint leg6_joint_roll: limit lower=-0.7854 upper=1.3090 effort=300 velocity=1 -> lower=-0.7854 upper=1.3090 effort=300 velocity=3
- joint leg6_joint_stick: axis 0 0 1 -> 1 1 1; limit lower=-0.01 upper=0.01 effort=300 velocity=1 -> lower=-0.08 upper=0.08 effort=300 velocity=1

Commit message: 修改模型

File: urdf/new_hexapod.urdf (robot description, URDF)
Before this commit: robot hexapod, 31 links, 30 joints
Links:
- link leg1_pitch_3: mass 0.275 -> 0.245; geometry collision cylinder length=0.125 radius=0.025; visual cylinder length=0.125 radius=0.025
- link leg1_stick: mass 0.133 -> 0.15; geometry collision sphere radius=0.025; visual sphere radius=0.025
- link leg2_pitch_3: mass 0.275 -> 0.245; geometry collision cylinder length=0.125 radius=0.025; visual cylinder length=0.125 radius=0.025
- link leg2_stick: mass 0.133 -> 0.15; geometry collision sphere radius=0.025; visual sphere radius=0.025
- link leg3_pitch_3: mass 0.275 -> 0.245; geometry collision cylinder length=0.125 radius=0.025; visual cylinder length=0.125 radius=0.025
- link leg3_stick: mass 0.133 -> 0.15; geometry collision sphere radius=0.025; visual sphere radius=0.025
- link leg4_pitch_3: mass 0.275 -> 0.245; geometry collision cylinder length=0.125 radius=0.025; visual cylinder length=0.125 radius=0.025
- link leg4_stick: mass 0.133 -> 0.15; geometry collision sphere radius=0.025; visual sphere radius=0.025
- link leg5_pitch_3: mass 0.275 -> 0.245; geometry collision cylinder length=0.125 radius=0.025; visual cylinder length=0.125 radius=0.025
- link leg5_stick: mass 0.133 -> 0.15; geometry collision sphere radius=0.025; visual sphere radius=0.025
- link leg6_pitch_3: mass 0.275 -> 0.245; geometry collision cylinder length=0.125 radius=0.025; visual cylinder length=0.125 radius=0.025
- link leg6_stick: mass 0.133 -> 0.15; geometry collision sphere radius=0.025; visual sphere radius=0.025
Joints:
- joint leg1_joint_stick: axis 1 1 1 -> (none); limit lower=-0.08 upper=0.08 effort=300 velocity=1 -> (none); origin xyz=0.14 0 0 rpy=0 0 0 -> xyz=0.125 0 0 rpy=0 0 0; type revolute -> fixed
- joint leg2_joint_stick: axis 1 1 1 -> (none); limit lower=-0.08 upper=0.08 effort=300 velocity=1 -> (none); origin xyz=0.14 0 0 rpy=0 0 0 -> xyz=0.125 0 0 rpy=0 0 0; type revolute -> fixed
- joint leg3_joint_stick: axis 1 1 1 -> (none); limit lower=-0.08 upper=0.08 effort=300 velocity=1 -> (none); origin xyz=0.14 0 0 rpy=0 0 0 -> xyz=0.125 0 0 rpy=0 0 0; type revolute -> fixed
- joint leg4_joint_stick: axis 1 1 1 -> (none); limit lower=-0.08 upper=0.08 effort=300 velocity=1 -> (none); origin xyz=0.14 0 0 rpy=0 0 0 -> xyz=0.125 0 0 rpy=0 0 0; type revolute -> fixed
- joint leg5_joint_stick: axis 1 1 1 -> (none); limit lower=-0.08727 upper=0.08727 effort=300 velocity=1 -> (none); origin xyz=0.14 0 0 rpy=0 0 0 -> xyz=0.125 0 0 rpy=0 0 0; type revolute -> fixed
- joint leg6_joint_stick: axis 1 1 1 -> (none); limit lower=-0.08 upper=0.08 effort=300 velocity=1 -> (none); origin xyz=0.14 0 0 rpy=0 0 0 -> xyz=0.125 0 0 rpy=0 0 0; type revolute -> fixed
